File: ArduinoMega-24V-with-CH340.sch (KiCad schematic (older format))
At the start: 63 parts, among them IC1 ATMEGA2560-16AU, J1 BARREL_JACK, J10 CONN_01X04, J11 Mount, J12 Mount, J13 Mount, J14 Mount, J15 Mount, J16 Mount, J2 CONN_02X18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

Commit message: kicad5 windows version
Parts:
- C1, C14, C9: symbol device:CP_Small -> ArduinoMega-24V-with-CH340-rescue:CP_Small-device
- C10, C11, C12, C13, C15, C16, C17, C18, C2, C3, C4, C5, C6, C7, C8: symbol device:C_Small -> ArduinoMega-24V-with-CH340-rescue:C_Small-device
- D1: symbol device:D_Zener_Small -> ArduinoMega-24V-with-CH340-rescue:D_Zener_Small-device
- D2: symbol device:D -> ArduinoMega-24V-with-CH340-rescue:D-device
- D7: symbol device:D_Small -> ArduinoMega-24V-with-CH340-rescue:D_Small-device
- L1: symbol device:L_Small -> ArduinoMega-24V-with-CH340-rescue:L_Small-device
- Q1: symbol device:Q_PMOS_GDS -> ArduinoMega-24V-with-CH340-rescue:Q_PMOS_GDS-device
- R1, R2, R4, R5, R6, R7, R8: symbol device:R -> ArduinoMega-24V-with-CH340-rescue:R-device
- R10, R11, R3, R9: symbol device:R_Small -> ArduinoMega-24V-with-CH340-rescue:R_Small-device
- U1: symbol linear:LMV358 -> ArduinoMega-24V-with-CH340-rescue:LMV358-linear
- Y1, Y2: symbol device:Crystal_Small -> ArduinoMega-24V-with-CH340-rescue:Crystal_Small-device
